File: PCB/PUBG_KEY/PUBG_KEY.kicad_pcb (KiCad board)
At the start: 2 copper layers, 55 x 30 mm, 30 parts, among them J3 KEY_IN, U1 CH32V203F6P6, U2 AMS1117-3.3, Y1 8MHz

Commit message: update 19.04.2025
Other:
- outline, holes or cut-outs redrawn
- board text added: "KEY1"
- board text added: "KEY2"
- board text added: "KEY3"
- board text added: "KEY4"
- board text added: "https://github.com/Solderingironspb/Keyboard-for-PUBG"
Changed lines of the file:
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@@
 		(allow_soldermask_bridges_in_footprints no)
 		(pcbplotparams
-			(layerselection 0x00010fc_ffffffff)
+			(layerselection 0x003ffff_ffffffff)
 			(plot_on_all_layers_selection 0x0000000_00000000)
 			(disableapertmacros no)
@@
 			(outputformat 1)
 			(mirror no)
-			(drillshape 1)
+			(drillshape 0)
 			(scaleselection 1)
-			(outputdirectory "")
+			(outputdirectory "Gerber/")
 		)
 	)
@@
 		(tags "capacitor")
 		(property "Reference" "C4"
-			(at 0 -1.43 90)
+			(at 2.1 0.05 180)
 			(layer "F.SilkS")
 			(effects
@@
 		(tags "capacitor")
 		(property "Reference" "C7"
-			(at 0 -1.43 0)
+			(at 0.165 1.31 0)
 			(layer "F.SilkS")
 			(effects
@@
 		(tags "resistor")
 		(property "Reference" "R2"
-			(at 0 -1.65 0)
+			(at 0 -4.77 0)
 			(layer "F.SilkS")
 			(effects
@@
 		(tags "resistor")
 		(property "Reference" "R4"
-			(at 0 -1.65 0)
+			(at 0 -3.77 0)
 			(layer "F.SilkS")
 			(effects
@@
 		(tags "resistor")
 		(property "Reference" "R3"
-			(at 0 -1.65 0)
+			(at 0 -5.77 0)
 			(layer "F.SilkS")
 			(effects
@@
 		(tags "capacitor tantalum")
 		(property "Reference" "C2"
-			(at -3.64 -0.03 90)
+			(at -3.64 -0.03 180)
 			(layer "B.SilkS")
 			(effects
@@
 		(tags "CMS SOT")
 		(property "Reference" "U2"
-			(at 0 4.5 90)
+			(at 0 0.2 90)
 			(layer "B.SilkS")
 			(effects
@@
 		(tags "capacitor tantalum")
 		(property "Reference" "C1"
-			(at -3.52 0.33 90)
+			(at -3.52 0.33 180)
 			(layer "B.SilkS")
 			(effects
@@
 		(tags "capacitor")
 		(property "Reference" "C8"
-			(at 0 1.43 90)
+			(at 2.265 0.02 180)
 			(layer "B.SilkS")
 			(effects
@@
 		(tags "capacitor")
 		(property "Reference" "C5"
-			(at 0 1.825 0)
+			(at -0.87 1.825 0)
 			(layer "B.SilkS")
 			(effects
@@
 	)
 	(gr_circle
-		(center 78.03 81.67)
-		(end 78.04 81.67)
-		(stroke
-			(width 0.0001)
-			(type default)
-		)
-		(fill solid)
-		(layer "Edge.Cuts")
-	)
-	(gr_circle
 		(center 102.53 69.67)
 		(end 104.03 69.67)
@@
 		(layer "Edge.Cuts")
 	)
+	(gr_text "https://github.com/Solderingironspb/Keyboard-for-PUBG"
+		(at 103.5 84.5 0)
+		(layer "B.SilkS")
+		(effects
+			(font
+				(size 0.8 0.8)
+				(thickness 0.125)
+			)
+			(justify left bottom mirror)
+		)
+	)
+	(gr_text "KEY4"
+		(at 89.497143 94 0)
+		(layer "B.SilkS")
+		(effects
+			(font
+				(size 1 1)
+				(thickness 0.1)
+			)
+			(justify left bottom mirror)
+		)
+	)
+	(gr_text "GND\n"
+		(at 84.08381 94 0)
+		(layer "B.SilkS")
+		(effects
+			(font
+				(size 1 1)
+				(thickness 0.1)
+			)
+			(justify left bottom mirror)
+		)
+	)
+	(gr_text "KEY3\n"
+		(at 79.337143 94 0)
+		(layer "B.SilkS")
+		(effects
+			(font
+				(size 1 1)
+				(thickness 0.1)
+			)
+			(justify left bottom mirror)
+		)
+	)
+	(gr_text "GND\n"
+		(at 68.84381 94 0)
+		(layer "B.SilkS")
+		(effects
+			(font
+				(size 1 1)
+				(thickness 0.1)
+			)
+			(justify left bottom mirror)
+		)
+	)
+	(gr_text "KEY2"
+		(at 74.257143 94 0)
+		(layer "B.SilkS")
+		(effects
+			(font
+				(size 1 1)
+				(thickness 0.1)
+			)
+			(justify left bottom mirror)
+		)
+	)
+	(gr_text "KEY1\n"
+		(at 64.097143 94 0)
+		(layer "B.SilkS")
+		(effects
+			(font
+				(size 1 1)
+				(thickness 0.1)
+			)
+			(justify left bottom mirror)
+		)
+	)
 	(gr_text "Volkov Oleg\n2025"
 		(at 56.5 75 90)
@@
 	)
 	(group ""
-		(members "03438cd7-189b-4cc6-ad4d-1efeba951294" "15692789-3d00-4a18-9b59-dd247f2ffd1a"
-			"2b2ad4fb-2674-4ae6-9f89-962903ee67d6" "3ec32983-ef2f-456f-8b8c-856b6ba8262f"
-			"510e4d58-e36d-4c35-ae76-5333bafa24ac" "7159dedf-cefa-4532-a623-74d65e233c46"
-			"77890e66-0ce9-4987-891a-95dc6651cc00" "9c9e30d9-897a-4c26-96a0-111480837da1"
-			"b3bf6a2c-2cc1-4e62-83b9-d81f65f8fd56" "b4e83eb9-d012-4bf8-b6b4-275a244453a5"
-			"c3c6dc3d-35ba-4de2-b79c-6bb4e6b8e72b" "cf1ea56c-f089-4311-8a2f-9bc83b58490c"
-			"d4e1c6a3-3e1d-47bb-953b-dd33d73c1da9" "e107ca39-09bd-41c9-82ad-e41731e5411e"
-			"e3dce8ab-2360-4532-8561-0cc2b81ab44e" "eb97246c-305e-4506-99b9-cf617906fb98"
-			"f2b474c7-4dcf-4eeb-8e73-428a6b58649d"
+		(members "03438cd7-189b-4cc6-ad4d-1efeba951294" "2b2ad4fb-2674-4ae6-9f89-962903ee67d6"
+			"3ec32983-ef2f-456f-8b8c-856b6ba8262f" "510e4d58-e36d-4c35-ae76-5333bafa24ac"
+			"7159dedf-cefa-4532-a623-74d65e233c46" "77890e66-0ce9-4987-891a-95dc6651cc00"
+			"9c9e30d9-897a-4c26-96a0-111480837da1" "b3bf6a2c-2cc1-4e62-83b9-d81f65f8fd56"
+			"b4e83eb9-d012-4bf8-b6b4-275a244453a5" "c3c6dc3d-35ba-4de2-b79c-6bb4e6b8e72b"
+			"cf1ea56c-f089-4311-8a2f-9bc83b58490c" "d4e1c6a3-3e1d-47bb-953b-dd33d73c1da9"
+			"e107ca39-09bd-41c9-82ad-e41731e5411e" "e3dce8ab-2360-4532-8561-0cc2b81ab44e"
+			"eb97246c-305e-4506-99b9-cf617906fb98" "f2b474c7-4dcf-4eeb-8e73-428a6b58649d"
 		)
 	)
